Commit message: asdfasd

File: hydrone_aerial_underwater_description/urdf/hydrone_aerial_underwater_aerial.gazebo.xacro (robot description, xacro)
@@ -11,5 +11,5 @@
     <!-- <xacro:property name="volume" value="0.00001"/> -->
     <!-- <xacro:property name="volume" value="0.001"/> -->
-    <xacro:property name="volume" value="0.0001"/>
+    <xacro:property name="volume" value="0.00005"/>
     <!-- <xacro:property name="volume" value="0.00005"/> -->
     <xacro:property name="M_PI" value="3.1415926535897931" />
